File: Placa_TP2/Placa_TP2.kicad_pcb (KiCad board)
At the start: 2 copper layers, 70 x 70 mm, 0 parts

Commit message: mañana termino
Parts:
- added C1: 10n, Capacitor_THT:CP_Radial_D6.3mm_P2.50mm, F.Cu at (112.7, 77.4)
- added J1: Conn_01x02_Socket, Connector_Wire:SolderWire-0.1sqmm_1x02_P3.6mm_D0.4mm_OD1mm, F.Cu at (76.0, 93.4)
- added J2: Conn_01x02_Socket, Connector_Wire:SolderWire-0.1sqmm_1x02_P3.6mm_D0.4mm_OD1mm, F.Cu at (126.0, 83.2)
- added J3: Conn_01x02_Socket, Connector_Wire:SolderWire-0.1sqmm_1x02_P3.6mm_D0.4mm_OD1mm, F.Cu at (73.0, 67.3)
- added J4: Conn_01x02_Socket, Connector_Wire:SolderWire-0.1sqmm_1x02_P3.6mm_D0.4mm_OD1mm, F.Cu at (124.5, 63.7)
- added R1: 15k, Resistor_THT:R_Axial_DIN0204_L3.6mm_D1.6mm_P7.62mm_Horizontal, F.Cu at (89.2, 70.9)
- added R2: 1k, Resistor_THT:R_Axial_DIN0204_L3.6mm_D1.6mm_P7.62mm_Horizontal, F.Cu at (117.0, 62.2)
- added R3: 1k, Resistor_THT:R_Axial_DIN0204_L3.6mm_D1.6mm_P7.62mm_Horizontal, F.Cu at (107.5, 69.8)
- added R4: 1k, Resistor_THT:R_Axial_DIN0204_L3.6mm_D1.6mm_P7.62mm_Horizontal, F.Cu at (119.5, 101.5)
- added R5: 1k, Resistor_THT:R_Axial_DIN0204_L3.6mm_D1.6mm_P7.62mm_Horizontal, F.Cu at (87.5, 90.6)
- added R6: 90, Resistor_THT:R_Axial_DIN0204_L3.6mm_D1.6mm_P7.62mm_Horizontal, F.Cu at (80.5, 90.6)
- added R7: 1k, Resistor_THT:R_Axial_DIN0204_L3.6mm_D1.6mm_P7.62mm_Horizontal, F.Cu at (103.1, 100.9)
- added R8: 2700, Resistor_THT:R_Axial_DIN0204_L3.6mm_D1.6mm_P7.62mm_Horizontal, F.Cu at (103.3, 97.9)
- added R9: 51000, Resistor_THT:R_Axial_DIN0204_L3.6mm_D1.6mm_P7.62mm_Horizontal, F.Cu at (120.0, 81.5)
- added U1: TL084, Package_DIP:DIP-14_W7.62mm_Socket, F.Cu at (96.4, 78.8)
Routing:
- net GND: track 0.00 -> 84.6 mm
- net Net-(U1D--): track 0.00 -> 45.7 mm
- net /Vin: track 0.00 -> 35.6 mm
- net Net-(U1B--): track 0.00 -> 31.5 mm
- net Net-(U1B-+): track 0.00 -> 27.7 mm
- net /+Vcc: track 0.00 -> 26.7 mm, vias 0 -> 1
- net /Vout: track 0.00 -> 20.7 mm
- net Net-(U1A--): track 0.00 -> 17.8 mm
- net /-Vcc: track 0.00 -> 17.6 mm
- net Net-(U1C--): track 0.00 -> 16.5 mm
- net Net-(R7-Pad2): track 0.00 -> 13.1 mm
- net Net-(U1C-+): track 0.00 -> 12.8 mm

Commit message: placa final
Parts:
- moved R8 40.4 mm to (107.0, 57.7), turned to -90 degrees
- moved R6 30.5 mm to (106.5, 106.5), turned to 0 degrees
- moved R2 28.4 mm to (89.0, 57.5)
- moved R4 24.7 mm to (94.8, 100.5), turned to 180 degrees
- moved R5 21.4 mm to (106.7, 100.0), turned to 0 degrees
- moved R7 16.9 mm to (87.2, 106.5), turned to 0 degrees
- moved R3 13.3 mm to (95.0, 65.3)
- moved R1 10.4 mm to (80.5, 65.1), turned to 90 degrees
- moved J1 8.39 mm to (69.5, 88.1), turned to 90 degrees
- moved R9 7.83 mm to (121.5, 73.8)
- moved C1 6.51 mm to (114.0, 71.0), turned to 90 degrees
- moved J4 4.84 mm to (127.5, 67.5), turned to 90 degrees
- moved J2 3.00 mm to (129.0, 83.2)
Connections:
- R2 pad 2: Net-(U1C-+) -> Net-(U1B-+)
- R3 pad 2: Net-(U1C-+) -> Net-(U1B-+)
- R4 pad 1: Net-(U1B--) -> Net-(U1C--)
- R4 pad 2: Net-(U1C--) -> Net-(U1B--)
- R5 pad 2: Net-(U1B-+) -> Net-(U1C-+)
- R6 pad 1: Net-(U1B-+) -> Net-(U1C-+)
- R7 pad 1: Net-(U1C--) -> Net-(U1B--)
- U1 pad 7: Net-(U1B--) -> Net-(R7-Pad2)
- U1 pad 8: Net-(R7-Pad2) -> Net-(U1C--)
Routing:
- net GND: track 84.6 -> 179.7 mm
- net /+Vcc: track 26.7 -> 84.0 mm
- net Net-(R7-Pad2): track 13.1 -> 58.9 mm
- net /Vout: track 20.7 -> 59.8 mm
- net Net-(U1B-+): track 27.7 -> 44.6 mm
- net Net-(U1C-+): track 12.8 -> 29.0 mm
- net Net-(U1B--): track 31.5 -> 22.3 mm
- net /-Vcc: track 17.6 -> 25.1 mm
- net /Vin: track 35.6 -> 37.7 mm
- net Net-(U1D--): track 45.7 -> 43.9 mm
- net Net-(U1A--): track 17.8 -> 16.7 mm
- net Net-(U1C--): track 16.5 -> 15.5 mm
