File: Placa_TP2/Placa_TP2.kicad_sch (KiCad schematic)
At the start: 15 parts, among them J1 Conn_01x02_Socket, J2 Conn_01x02_Socket, J3 Conn_01x02_Socket, J4 Conn_01x02_Socket, U1 TL084

Commit message: mañana termino
Parts:
- C1: footprint Capacitor_THT:CP_Radial_D4.0mm_P1.50mm -> Capacitor_THT:CP_Radial_D6.3mm_P2.50mm
- J2, J4: footprint Connector_Wire:SolderWire-0.1sqmm_1x01_D0.4mm_OD1mm -> Connector_Wire:SolderWire-0.1sqmm_1x02_P3.6mm_D0.4mm_OD1mm
- R1, R2, R3, R4, R5, R6, R7, R8, R9: footprint Resistor_THT:R_Array_SIP4 -> Resistor_THT:R_Axial_DIN0204_L3.6mm_D1.6mm_P7.62mm_Horizontal
Other:
- moved on the sheet: R1, R4, U1C, U1D

Commit message: placa final
Connections:
- net at R7.2, R8.1: now also U1.7; no longer U1.8
- net at R5.2, R6.1: now also U1.10 (+); no longer U1.5 (+)
- net at R4.2, R7.1: now also U1.6 (-); no longer U1.9 (-)
- net at R2.2, R3.2: now also U1.5 (+); no longer U1.10 (+)
- new net: R4.1, U1.8, U1.9 (-)
Other:
- moved on the sheet: U1B, U1C
